File: Control_panel/Control_panel.kicad_pcb (KiCad board)
At the start: 2 copper layers, 196 parts, among them J1 Conn_02x32_Odd_Even, J2 Conn_01x02, J3 USB_B, SW1 SW_Push, SW10 SW_DIP_x08, SW11 SW_DIP_x08, SW2 SW_Push, SW3 SW_Push, SW4 SW_Push, SW5 SW_DIP_x08, SW6 SW_DIP_x08, SW7 SW_DIP_x08, SW8 SW_DIP_x08, SW9 SW_DIP_x08

Commit message: Register board and Control panel ordered
Parts:
- removed D4: LED, LED_SMD:LED_0603_1608Metric_Pad1.05x0.95mm_HandSolder
- removed J3: USB_B, Connector_USB:USB_B_OST_USB-B1HSxx_Horizontal
- removed R5: 330R, Resistor_SMD:R_0603_1608Metric_Pad0.98x0.95mm_HandSolder
- added H1: MountingHole, MountingHole:MountingHole_3.5mm, F.Cu at (98.0, 41.0)
- added H2: MountingHole, MountingHole:MountingHole_3.5mm, F.Cu at (214.0, 41.0)
- added H3: MountingHole, MountingHole:MountingHole_3.5mm, F.Cu at (98.0, 99.0)
- added H4: MountingHole, MountingHole:MountingHole_3.5mm, F.Cu at (214.0, 99.0)
- D1, D2, D3, D5, D6, D7, D8, D9: value LED -> YELLOW
- D10, D11, D12, D13, D14, D15, D16, D17, D18, D19, D20, D21, D22, D23, D24, D25, D26, D27, D28, D29, D30, D31, D32, D33: value LED -> RED
- D34, D35, D36, D37, D38, D39, D40, D41, D42, D43, D44, D45, D46, D47, D48, D49, D50, D51, D52, D53, D54, D55, D56, D57, D58, D59, D60, D61, D62, D63: value LED -> GREEN
- R100, R101, R102, R103, R108, R109, R110, R111, R116, R117, R118, R119, R15, R16, R17, R21, R22, R23, R27, R28, R29, R3, R33, R34, R35, R39, R40, R41, R45, R46, R47, R51, R52, R53, R57, R58, R59, R64, R65, R66, R67, R72, R73, R74, R75, R8, R80, R81, R82, R83, R87, R88, R89, R93, R94, R95: value 1K -> 10K
- moved D9 183.1 mm to (210.2, 53.3), turned to -90 degrees
- moved R7 180.6 mm to (210.2, 84.5), turned to -90 degrees
- moved R11 178.7 mm to (210.2, 57.1), turned to -90 degrees
- moved D6 178.5 mm to (210.2, 80.6), turned to -90 degrees
- moved R8 178.3 mm to (208.3, 84.5), turned to -90 degrees
- moved R14 170.1 mm to (201.3, 57.1), turned to -90 degrees
- moved D12 166.7 mm to (201.3, 53.3), turned to -90 degrees
- moved D15 165.0 mm to (198.8, 53.3), turned to -90 degrees
- moved D18 164.1 mm to (196.2, 53.3), turned to -90 degrees
- moved R23 163.4 mm to (198.8, 72.4), turned to 90 degrees
- moved R20 162.7 mm to (198.8, 57.1), turned to -90 degrees
- moved R26 160.2 mm to (196.2, 57.1), turned to -90 degrees
- moved R29 160.1 mm to (196.2, 72.4), turned to 90 degrees
- moved D37 156.7 mm to (201.3, 80.6), turned to 90 degrees
- moved R67 155.7 mm to (201.3, 99.7), turned to 90 degrees
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Connections:
- D1 pad 1: /~{RESET} -> Net-(D1-K)
- D1 pad 2: Net-(D1-A) -> +5V
- D2 pad 1: GND -> Net-(D2-K)
- D2 pad 2: Net-(D2-A) -> /CARRY_FLAG_A
- D3 pad 1: GND -> Net-(D3-K)
- D3 pad 2: Net-(D3-A) -> /EQUAL_FLAG_A
- D5 pad 1: GND -> Net-(D5-K)
- D5 pad 2: Net-(D5-A) -> /CARRY_FLAG_B
- D7 pad 1: GND -> Net-(D7-K)
- D7 pad 2: Net-(D7-A) -> /EQUAL_FLAG_B
- R1 pad 1: Net-(D1-A) -> /~{RESET}
- R1 pad 2: +5V -> Net-(D1-K)
- R2 pad 1: Net-(D2-A) -> GND
- R2 pad 2: /CARRY_FLAG_A -> Net-(D2-K)
- R4 pad 1: Net-(D3-A) -> GND
- R4 pad 2: /EQUAL_FLAG_A -> Net-(D3-K)
- R6 pad 1: Net-(D5-A) -> GND
- R6 pad 2: /CARRY_FLAG_B -> Net-(D5-K)
- R9 pad 1: Net-(D7-A) -> GND
- R9 pad 2: /EQUAL_FLAG_B -> Net-(D7-K)
Routing:
- net +5V: track 0.00 -> 395.2 mm, vias 0 -> 2
- net /CLK: track 0.00 -> 162.2 mm
- net /CONTROL_DISABLE: track 0.00 -> 120.7 mm, vias 0 -> 2
- net /~{PC_OUT}: track 0.00 -> 116.0 mm, vias 0 -> 1
- net /~{RESET}: track 0.00 -> 115.8 mm
- net /~{RAM_OUT}: track 0.00 -> 114.6 mm
- net /~{SP_OUT}: track 0.00 -> 112.6 mm, vias 0 -> 1
- net /~{ADR_H_OUT}: track 0.00 -> 110.2 mm, vias 0 -> 1
- net /~{A_OUT}: track 0.00 -> 108.9 mm, vias 0 -> 1
- net /~{ADR_L_OUT}: track 0.00 -> 99.1 mm, vias 0 -> 2
- net /~{BC_OUT}: track 0.00 -> 98.4 mm
- net /ALU_S0: track 0.00 -> 97.6 mm
- net /~{T_OUT}: track 0.00 -> 95.8 mm, vias 0 -> 1
- net /~{DE_OUT}: track 0.00 -> 94.9 mm
- net /~{ALU_OUT}: track 0.00 -> 94.9 mm, vias 0 -> 1
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- added copper zone on B.Cu, net GND
- added copper zone on F.Cu, net GND
Other:
- board outline added: 124 x 66 mm
- board text added: "A0"
- board text added: "A1"
- board text added: "A10"
- board text added: "A11"
- board text added: "A12"
- board text added: "A13"
- board text added: "A14"
- board text added: "A15"
- board text added: "A2"
- board text added: "A3"
- board text added: "A4"
- board text added: "A5"
- board text added: "A6"
- board text added: "A7"
- board text added: "A8"
- board text added: "A9"
- board text added: "AH OE"
- board text added: "AL OE"
- board text added: "ALU C"
- board text added: "ALU M"
- board text added: "ALU OE"
- board text added: "ALU S0"
- board text added: "ALU S1"
- board text added: "ALU S2"
- board text added: "ALU S3"
- board text added: "Acc OE"
- board text added: "Acc WE"
- board text added: "Address"
- board text added: "B WE"
- board text added: "BC OE"
- board text added: "C WE"
- board text added: "CONTROL PANEL"
- board text added: "Carry"
- board text added: "Clock"
- board text added: "D WE"
- board text added: "D0"
- board text added: "D1"
- board text added: "D2"
- board text added: "D3"
- board text added: "D4"
- board text added: "D5"
- board text added: "D6"
- board text added: "D7"
- board text added: "DE OE"
- board text added: "Data"
- board text added: "E WE"
- board text added: "Ed Atkinson 2023"
- board text added: "Equal"
- board text added: "FS WE"
- board text added: "FU WE"
- board text added: "Mem OE"
- board text added: "Mem WE"
- board text added: "PC OE"
- board text added: "PCH WE"
- board text added: "PCL WE"
- board text added: "Release"
- board text added: "Reset"
- board text added: "SP OE"
- board text added: "SPH WE"
- board text added: "SPL WE"
- board text added: "System"
- board text added: "T OUT"
- board text added: "T WE"
- board text added: "User"
