File: Control_panel/Control_panel.kicad_sch (KiCad schematic)
At the start: 196 parts, among them J1 Conn_02x32_Odd_Even, J2 Conn_01x02, J3 USB_B, SW1 SW_Push, SW10 SW_DIP_x08, SW11 SW_DIP_x08, SW2 SW_Push, SW3 SW_Push, SW4 SW_Push, SW5 SW_DIP_x08, SW6 SW_DIP_x08, SW7 SW_DIP_x08, SW8 SW_DIP_x08, SW9 SW_DIP_x08

Commit message: Register board and Control panel ordered
Parts:
- removed D4: LED, LED_SMD:LED_0603_1608Metric_Pad1.05x0.95mm_HandSolder, symbol Device:LED
- removed J3: USB_B, Connector_USB:USB_B_OST_USB-B1HSxx_Horizontal, symbol Connector:USB_B
- removed R5: 330R, Resistor_SMD:R_0603_1608Metric_Pad0.98x0.95mm_HandSolder, symbol Device:R
- added H1, H2, H3, H4: MountingHole, MountingHole:MountingHole_3.5mm, symbol Mechanical:MountingHole
- D1, D2, D3, D5, D6, D7, D8, D9: value LED -> YELLOW
- D10, D11, D12, D13, D14, D15, D16, D17, D18, D19, D20, D21, D22, D23, D24, D25, D26, D27, D28, D29, D30, D31, D32, D33: value LED -> RED
- D34, D35, D36, D37, D38, D39, D40, D41, D42, D43, D44, D45, D46, D47, D48, D49, D50, D51, D52, D53, D54, D55, D56, D57, D58, D59, D60, D61, D62, D63: value LED -> GREEN
- R100, R101, R102, R103, R108, R109, R110, R111, R116, R117, R118, R119, R15, R16, R17, R21, R22, R23, R27, R28, R29, R3, R33, R34, R35, R39, R40, R41, R45, R46, R47, R51, R52, R53, R57, R58, R59, R64, R65, R66, R67, R72, R73, R74, R75, R8, R80, R81, R82, R83, R87, R88, R89, R93, R94, R95: value 1K -> 10K
Connections:
- net +5V: now also D1.2 (A); no longer R1.2
- net CARRY_FLAG_A: now also D2.2 (A); no longer R2.2
- net CARRY_FLAG_B: now also D5.2 (A); no longer R6.2
- net EQUAL_FLAG_A: now also D3.2 (A); no longer R4.2
- net EQUAL_FLAG_B: now also D7.2 (A); no longer R9.2
- net GND: now also R2.1, R4.1, R6.1, R9.1; no longer D2.1 (K), D3.1 (K), D5.1 (K), D7.1 (K)
- net ~{RESET}: now also R1.1; no longer D1.1 (K)
- new net: D5.1 (K), R6.2
- new net: D2.1 (K), R2.2
- new net: D3.1 (K), R4.2
- new net: D7.1 (K), R9.2
- new net: D1.1 (K), R1.2
- no-connect marks 8 -> 6
Other:
- moved on the sheet: D1, D2, D3, D5, D7
