File: Register_board/Register_board.kicad_pcb (KiCad board)
At the start: 2 copper layers, 118 parts, among them J1 Conn_02x30_Odd_Even, U1 74LS374, U10 74LS244, U11 74LS194, U12 74LS181, U13 74LS181, U14 74LS194, U15 74LS244, U18 74LS77, U2 74LS374, U3 74LS374, U4 74LS374, U5 74LS374, U6 74LS374, U7 74LS374, U8 74LS374, U9 74LS244

Commit message: Register board schematic
Parts:
- removed U11, U14: 74LS194, Package_DIP:DIP-16_W7.62mm_Socket
- removed U12, U13: 74LS181, Package_DIP:DIP-24_W7.62mm_Socket
- removed U15: 74LS244, Package_DIP:DIP-20_W7.62mm_Socket
- removed U18: 74LS77, Package_DIP:DIP-12_W7.62mm_Socket
- added C16: 100nF, Capacitor_SMD:C_0603_1608Metric_Pad1.08x0.95mm_HandSolder, F.Cu at (169.0, 63.1)
- added D30: LED, LED_SMD:LED_0603_1608Metric_Pad1.05x0.95mm_HandSolder, F.Cu at (169.1, 83.2)
- added D31: LED, LED_SMD:LED_0603_1608Metric_Pad1.05x0.95mm_HandSolder, F.Cu at (169.1, 85.8)
- added D32: LED, LED_SMD:LED_0603_1608Metric_Pad1.05x0.95mm_HandSolder, F.Cu at (169.1, 88.4)
- added D33: LED, LED_SMD:LED_0603_1608Metric_Pad1.05x0.95mm_HandSolder, F.Cu at (169.1, 91.0)
- added D34: LED, LED_SMD:LED_0603_1608Metric_Pad1.05x0.95mm_HandSolder, F.Cu at (169.1, 93.6)
- added D35: LED, LED_SMD:LED_0603_1608Metric_Pad1.05x0.95mm_HandSolder, F.Cu at (169.1, 96.1)
- added R58: 10K, Resistor_SMD:R_0603_1608Metric_Pad0.98x0.95mm_HandSolder, F.Cu at (169.0, 65.6)
- added R59: 10K, Resistor_SMD:R_0603_1608Metric_Pad0.98x0.95mm_HandSolder, F.Cu at (169.0, 68.1)
- added R60: 10K, Resistor_SMD:R_0603_1608Metric_Pad0.98x0.95mm_HandSolder, F.Cu at (169.0, 70.6)
- added R61: 10K, Resistor_SMD:R_0603_1608Metric_Pad0.98x0.95mm_HandSolder, F.Cu at (169.0, 73.1)
- added R62: 10K, Resistor_SMD:R_0603_1608Metric_Pad0.98x0.95mm_HandSolder, F.Cu at (169.0, 75.6)
- added R63: 10K, Resistor_SMD:R_0603_1608Metric_Pad0.98x0.95mm_HandSolder, F.Cu at (169.0, 78.1)
- added R64: 10K, Resistor_SMD:R_0603_1608Metric_Pad0.98x0.95mm_HandSolder, F.Cu at (169.0, 80.6)
- added R65: 10K, Resistor_SMD:R_0603_1608Metric_Pad0.98x0.95mm_HandSolder, F.Cu at (173.4, 63.1)
- added R66: 10K, Resistor_SMD:R_0603_1608Metric_Pad0.98x0.95mm_HandSolder, F.Cu at (173.4, 65.6)
- added R67: 10K, Resistor_SMD:R_0603_1608Metric_Pad0.98x0.95mm_HandSolder, F.Cu at (173.4, 68.1)
- added R68: 10K, Resistor_SMD:R_0603_1608Metric_Pad0.98x0.95mm_HandSolder, F.Cu at (173.4, 70.6)
- added R69: 10K, Resistor_SMD:R_0603_1608Metric_Pad0.98x0.95mm_HandSolder, F.Cu at (173.4, 73.1)
- added R70: 10K, Resistor_SMD:R_0603_1608Metric_Pad0.98x0.95mm_HandSolder, F.Cu at (173.4, 75.6)
- added R71: 10K, Resistor_SMD:R_0603_1608Metric_Pad0.98x0.95mm_HandSolder, F.Cu at (173.4, 78.1)
- added R72: 10K, Resistor_SMD:R_0603_1608Metric_Pad0.98x0.95mm_HandSolder, F.Cu at (173.4, 80.6)
- added R73: 10K, Resistor_SMD:R_0603_1608Metric_Pad0.98x0.95mm_HandSolder, F.Cu at (177.7, 63.1)
- added R74: 10K, Resistor_SMD:R_0603_1608Metric_Pad0.98x0.95mm_HandSolder, F.Cu at (177.7, 65.6)
- added R75: 10K, Resistor_SMD:R_0603_1608Metric_Pad0.98x0.95mm_HandSolder, F.Cu at (177.7, 68.1)
- added R76: 10K, Resistor_SMD:R_0603_1608Metric_Pad0.98x0.95mm_HandSolder, F.Cu at (177.7, 70.6)
- added R77: 10K, Resistor_SMD:R_0603_1608Metric_Pad0.98x0.95mm_HandSolder, F.Cu at (177.7, 73.1)
- added R78: 10K, Resistor_SMD:R_0603_1608Metric_Pad0.98x0.95mm_HandSolder, F.Cu at (177.7, 75.6)
- added R79: 10K, Resistor_SMD:R_0603_1608Metric_Pad0.98x0.95mm_HandSolder, F.Cu at (177.7, 78.1)
- added R80: 10K, Resistor_SMD:R_0603_1608Metric_Pad0.98x0.95mm_HandSolder, F.Cu at (177.7, 80.6)
- added R81: 10K, Resistor_SMD:R_0603_1608Metric_Pad0.98x0.95mm_HandSolder, F.Cu at (182.1, 63.1)
- added R82: 10K, Resistor_SMD:R_0603_1608Metric_Pad0.98x0.95mm_HandSolder, F.Cu at (182.1, 65.6)
- added R83: 10K, Resistor_SMD:R_0603_1608Metric_Pad0.98x0.95mm_HandSolder, F.Cu at (182.1, 68.1)
- added R84: 10K, Resistor_SMD:R_0603_1608Metric_Pad0.98x0.95mm_HandSolder, F.Cu at (182.1, 70.6)
- added R85: 10K, Resistor_SMD:R_0603_1608Metric_Pad0.98x0.95mm_HandSolder, F.Cu at (182.1, 73.1)
- added R86: 10K, Resistor_SMD:R_0603_1608Metric_Pad0.98x0.95mm_HandSolder, F.Cu at (182.1, 75.6)
- added R87: 10K, Resistor_SMD:R_0603_1608Metric_Pad0.98x0.95mm_HandSolder, F.Cu at (182.1, 78.1)
- added R88: 10K, Resistor_SMD:R_0603_1608Metric_Pad0.98x0.95mm_HandSolder, F.Cu at (182.1, 80.6)
- added R89: 10K, Resistor_SMD:R_0603_1608Metric_Pad0.98x0.95mm_HandSolder, F.Cu at (186.4, 63.1)
- added R90: 10K, Resistor_SMD:R_0603_1608Metric_Pad0.98x0.95mm_HandSolder, F.Cu at (186.4, 65.6)
- added R91: 10K, Resistor_SMD:R_0603_1608Metric_Pad0.98x0.95mm_HandSolder, F.Cu at (186.4, 68.1)
- added R92: 10K, Resistor_SMD:R_0603_1608Metric_Pad0.98x0.95mm_HandSolder, F.Cu at (186.4, 70.6)
- added R93: 10K, Resistor_SMD:R_0603_1608Metric_Pad0.98x0.95mm_HandSolder, F.Cu at (186.4, 73.1)
- added R94: 10K, Resistor_SMD:R_0603_1608Metric_Pad0.98x0.95mm_HandSolder, F.Cu at (186.4, 75.6)
- added R95: 10K, Resistor_SMD:R_0603_1608Metric_Pad0.98x0.95mm_HandSolder, F.Cu at (186.4, 78.1)
- added R96: 10K, Resistor_SMD:R_0603_1608Metric_Pad0.98x0.95mm_HandSolder, F.Cu at (186.4, 80.6)
- added U16: 74LS75, Package_DIP:DIP-16_W7.62mm_Socket, F.Cu at (157.2, 63.9)
- R14, R15, R30, R31, R32, R33, R34, R35: value 330R -> 10K
- R17, R18, R19, R20, R22, R23, R44, R45, R46, R47, R48, R49, R50, R51: value 10K -> 330R
Connections:
- D10 pad 2: /C_LOAD -> /B_LOAD
- D11 pad 1: /~{DE_OUT} -> Net-(D11-K)
- D11 pad 2: Net-(D11-A) -> /C_LOAD
- D14 pad 1: /~{ADR_H_OUT} -> /~{A_OUT}
- D15 pad 1: /~{ADR_L_OUT} -> /~{T_OUT}
- D16 pad 2: /ACC_S0 -> /A_LOAD
- D17 pad 2: /ACC_S1 -> /T_LOAD
- D18 pad 1: Net-(D18-K) -> /~{ADR_H_OUT}
- D18 pad 2: /ALU_S0 -> Net-(D18-A)
- D19 pad 1: Net-(D19-K) -> /~{ADR_L_OUT}
- D19 pad 2: /ALU_S1 -> Net-(D19-A)
- D20 pad 2: /ALU_S2 -> /ALU_S0
- D21 pad 2: /ALU_S3 -> /ALU_S1
- D22 pad 2: /ALU_M -> /ALU_S0
- D23 pad 1: /~{FLAGS_A_UPDATE} -> Net-(D23-K)
- D23 pad 2: Net-(D23-A) -> /ALU_S1
- D24 pad 1: /~{FLAGS_B_UPDATE} -> Net-(D24-K)
- D24 pad 2: Net-(D24-A) -> /ALU_S2
- D25 pad 1: /~{ALU_CIN} -> Net-(D25-K)
- D25 pad 2: Net-(D25-A) -> /ALU_S3
- D26 pad 1: Net-(D26-K) -> /~{ALU_CIN}
- D26 pad 2: /CARRY_FLAG_A -> Net-(D26-A)
- D27 pad 1: Net-(D27-K) -> /FLAGS_A_UPDATE
- D27 pad 2: /EQUAL_FLAG_A -> Net-(D27-A)
- D28 pad 1: Net-(D28-K) -> /FLAGS_B_UPDATE
- D28 pad 2: /CARRY_FLAG_B -> Net-(D28-A)
- D29 pad 2: /EQUAL_FLAG_B -> /ALU_M
- D3 pad 1: Net-(D3-K) -> /~{SP_OUT}
- D3 pad 2: /PC_H_LOAD -> Net-(D3-A)
- D4 pad 2: /PC_L_LOAD -> /PC_H_LOAD
- D5 pad 1: /~{SP_OUT} -> Net-(D5-K)
- D5 pad 2: Net-(D5-A) -> /PC_L_LOAD
- D9 pad 1: Net-(D9-K) -> /~{DE_OUT}
- D9 pad 2: /B_LOAD -> Net-(D9-A)
- J1 pad 26: unconnected-(J1-Pin_26-Pad26) -> /ALU_S0
- J1 pad 28: unconnected-(J1-Pin_28-Pad28) -> /ALU_S1
- J1 pad 30: unconnected-(J1-Pin_30-Pad30) -> /ALU_S2
- J1 pad 32: unconnected-(J1-Pin_32-Pad32) -> /ALU_S3
- J1 pad 34: unconnected-(J1-Pin_34-Pad34) -> /ALU_M
- J1 pad 36: unconnected-(J1-Pin_36-Pad36) -> /~{ALU_CIN}
- J1 pad 38: unconnected-(J1-Pin_38-Pad38) -> /FLAGS_A_UPDATE
- J1 pad 40: unconnected-(J1-Pin_40-Pad40) -> /FLAGS_B_UPDATE
- J1 pad 42: unconnected-(J1-Pin_42-Pad42) -> /CARRY_FLAG_A
- J1 pad 44: unconnected-(J1-Pin_44-Pad44) -> /EQUAL_FLAG_A
- J1 pad 46: unconnected-(J1-Pin_46-Pad46) -> /CARRY_FLAG_B
- J1 pad 48: unconnected-(J1-Pin_48-Pad48) -> /EQUAL_FLAG_B
- J1 pad 50: unconnected-(J1-Pin_50-Pad50) -> /A_LOAD
- J1 pad 52: unconnected-(J1-Pin_52-Pad52) -> /T_LOAD
- J1 pad 53: unconnected-(J1-Pin_53-Pad53) -> /~{A_OUT}
- J1 pad 54: unconnected-(J1-Pin_54-Pad54) -> /~{ALU_OUT}
- J1 pad 55: unconnected-(J1-Pin_55-Pad55) -> /~{T_OUT}
- J1 pad 57: /RESET -> /~{RESET}
- R11 pad 1: Net-(D11-A) -> Net-(D11-K)
- R11 pad 2: +5V -> GND
- R14 pad 1: Net-(D14-A) -> GND
- R14 pad 2: +5V -> /A0
- R15 pad 1: Net-(D15-A) -> GND
- R15 pad 2: +5V -> /A1
- R16 pad 1: /PC_H_LOAD -> GND
- R16 pad 2: GND -> /A2
- R17 pad 1: /PC_L_LOAD -> Net-(D14-A)
- R17 pad 2: GND -> +5V
- R18 pad 1: /SP_H_LOAD -> Net-(D15-A)
- R18 pad 2: GND -> +5V
- R19 pad 1: /SP_L_LOAD -> Net-(D16-K)
- R20 pad 1: /B_LOAD -> Net-(D17-K)
- R21 pad 1: /C_LOAD -> GND
- R21 pad 2: GND -> /A3
- R22 pad 1: /D_LOAD -> Net-(D18-A)
- R22 pad 2: GND -> +5V
- R23 pad 1: /E_LOAD -> Net-(D19-A)
- R23 pad 2: GND -> +5V
- R24 pad 1: /RESET -> GND
- R24 pad 2: GND -> /A4
- R25 pad 1: /CLK -> GND
- R25 pad 2: GND -> /A5
- R26 pad 1: /~{PC_OUT} -> GND
- R26 pad 2: +5V -> /A6
- R27 pad 1: /~{SP_OUT} -> GND
- R27 pad 2: +5V -> /A7
- R28 pad 1: /~{BC_OUT} -> GND
- R28 pad 2: +5V -> /A8
- R29 pad 1: /~{DE_OUT} -> GND
- R29 pad 2: +5V -> /A9
- R3 pad 1: Net-(D3-K) -> Net-(D3-A)
- R3 pad 2: GND -> +5V
- R30 pad 1: Net-(D16-K) -> GND
- R30 pad 2: GND -> /A10
- R31 pad 1: Net-(D17-K) -> GND
- R31 pad 2: GND -> /A11
- R32 pad 1: Net-(D18-K) -> GND
- R32 pad 2: GND -> /A12
- R33 pad 1: Net-(D19-K) -> GND
- R33 pad 2: GND -> /A13
- R34 pad 1: Net-(D20-K) -> GND
- R34 pad 2: GND -> /A14
- R35 pad 1: Net-(D21-K) -> GND
- R35 pad 2: GND -> /A15
- R36 pad 1: Net-(D22-K) -> Net-(D20-K)
- R37 pad 1: Net-(D23-A) -> Net-(D21-K)
- R37 pad 2: +5V -> GND
- R38 pad 1: Net-(D24-A) -> Net-(D22-K)
- R38 pad 2: +5V -> GND
- R39 pad 1: Net-(D25-A) -> Net-(D23-K)
- R39 pad 2: +5V -> GND
- R40 pad 1: Net-(D26-K) -> Net-(D24-K)
- R41 pad 1: Net-(D27-K) -> Net-(D25-K)
- R42 pad 1: Net-(D28-K) -> Net-(D26-A)
- R42 pad 2: GND -> +5V
- R43 pad 1: Net-(D29-K) -> Net-(D27-A)
- R43 pad 2: GND -> +5V
- R44 pad 1: /~{ALU_CIN} -> Net-(D28-A)
- R45 pad 1: /~{FLAGS_A_UPDATE} -> Net-(D29-K)
- R45 pad 2: +5V -> GND
- R46 pad 1: /~{FLAGS_B_UPDATE} -> Net-(D30-K)
- R46 pad 2: +5V -> GND
- R47 pad 1: /ACC_S0 -> Net-(D31-A)
- R47 pad 2: GND -> +5V
- R48 pad 1: /ACC_S1 -> Net-(D32-K)
- R49 pad 1: /ALU_S0 -> Net-(D33-K)
- R5 pad 1: Net-(D5-A) -> Net-(D5-K)
- R5 pad 2: +5V -> GND
- R50 pad 1: /ALU_S1 -> Net-(D34-K)
- R51 pad 1: /ALU_S2 -> Net-(D35-K)
- R52 pad 1: /ALU_S3 -> GND
- R52 pad 2: GND -> /L0
- R53 pad 1: /ALU_M -> GND
- R53 pad 2: GND -> /D0
- R54 pad 1: /CARRY_FLAG_A -> GND
- R54 pad 2: GND -> /L1
- R55 pad 1: /EQUAL_FLAG_A -> GND
- R55 pad 2: GND -> /D1
- R56 pad 1: /CARRY_FLAG_B -> GND
- R56 pad 2: GND -> /L2
- R57 pad 1: /EQUAL_FLAG_B -> GND
- R57 pad 2: GND -> /D2
- R9 pad 1: Net-(D9-K) -> Net-(D9-A)
- R9 pad 2: GND -> +5V
- U1 pad 13: /D4 -> /ALU4
- U1 pad 14: /D5 -> /ALU5
- U1 pad 17: /D6 -> /ALU6
- U1 pad 18: /D7 -> /ALU7
- U1 pad 3: /D0 -> /ALU0
- U1 pad 4: /D1 -> /ALU1
- U1 pad 7: /D2 -> /ALU2
- U1 pad 8: /D3 -> /ALU3
- U10 pad 12: /D3 -> /L3
- U10 pad 14: /D2 -> /L2
- U10 pad 16: /D1 -> /L1
- U10 pad 18: /D0 -> /L0
- U10 pad 3: /D7 -> /L7
- U10 pad 5: /D6 -> /L6
- U10 pad 7: /D5 -> /L5
- U10 pad 9: /D4 -> /L4
- U2 pad 13: /D4 -> /ALU4
- U2 pad 14: /D5 -> /ALU5
- U2 pad 17: /D6 -> /ALU6
- U2 pad 18: /D7 -> /ALU7
- U2 pad 3: /D0 -> /ALU0
- U2 pad 4: /D1 -> /ALU1
- U2 pad 7: /D2 -> /ALU2
- U2 pad 8: /D3 -> /ALU3
- U3 pad 13: /D4 -> /ALU4
- U3 pad 14: /D5 -> /ALU5
- U3 pad 17: /D6 -> /ALU6
- U3 pad 18: /D7 -> /ALU7
- U3 pad 3: /D0 -> /ALU0
- U3 pad 4: /D1 -> /ALU1
- U3 pad 7: /D2 -> /ALU2
- U3 pad 8: /D3 -> /ALU3
- U4 pad 13: /D4 -> /ALU4
- U4 pad 14: /D5 -> /ALU5
- U4 pad 17: /D6 -> /ALU6
- U4 pad 18: /D7 -> /ALU7
- U4 pad 3: /D0 -> /ALU0
- U4 pad 4: /D1 -> /ALU1
- U4 pad 7: /D2 -> /ALU2
- U4 pad 8: /D3 -> /ALU3
- U5 pad 13: /D4 -> /ALU4
- U5 pad 14: /D5 -> /ALU5
- U5 pad 17: /D6 -> /ALU6
- U5 pad 18: /D7 -> /ALU7
- U5 pad 3: /D0 -> /ALU0
- U5 pad 4: /D1 -> /ALU1
- U5 pad 7: /D2 -> /ALU2
- U5 pad 8: /D3 -> /ALU3
- U6 pad 13: /D4 -> /ALU4
- U6 pad 14: /D5 -> /ALU5
- U6 pad 17: /D6 -> /ALU6
- U6 pad 18: /D7 -> /ALU7
- U6 pad 3: /D0 -> /ALU0
- U6 pad 4: /D1 -> /ALU1
- U6 pad 7: /D2 -> /ALU2
- U6 pad 8: /D3 -> /ALU3
- U7 pad 13: /D4 -> /ALU4
- U7 pad 14: /D5 -> /ALU5
- U7 pad 17: /D6 -> /ALU6
- U7 pad 18: /D7 -> /ALU7
- U7 pad 3: /D0 -> /ALU0
- U7 pad 4: /D1 -> /ALU1
- U7 pad 7: /D2 -> /ALU2
- U7 pad 8: /D3 -> /ALU3
- U8 pad 13: /D4 -> /ALU4
- U8 pad 14: /D5 -> /ALU5
- U8 pad 17: /D6 -> /ALU6
- U8 pad 18: /D7 -> /ALU7
- U8 pad 3: /D0 -> /ALU0
- U8 pad 4: /D1 -> /ALU1
- U8 pad 7: /D2 -> /ALU2
- U8 pad 8: /D3 -> /ALU3
- U9 pad 12: /D3 -> /L3
- U9 pad 14: /D2 -> /L2
- U9 pad 16: /D1 -> /L1
- U9 pad 18: /D0 -> /L0
- U9 pad 3: /D7 -> /L7
- U9 pad 5: /D6 -> /L6
- U9 pad 7: /D5 -> /L5
- U9 pad 9: /D4 -> /L4
Routing:
- net +5V: track 283.0 -> 139.8 mm
- net Net-(U12-A=B): track 102.8 -> 0.00 mm
- net /ALU_M: track 73.7 -> 0.00 mm
- net Net-(U11-Q0): track 62.2 -> 0.00 mm
- net Net-(U11-Dsl): track 55.1 -> 0.00 mm
- net Net-(U12-Cn+4): track 51.2 -> 0.00 mm
- net /D4: track 207.6 -> 164.1 mm, vias 1 -> 0
- net /CLK: track 40.9 -> 0.00 mm
- net /ACC_S1: track 37.9 -> 0.00 mm
- net /ALU_S0: track 36.9 -> 0.00 mm
- net Net-(U13-A0): track 35.8 -> 0.00 mm
- net /ALU_S1: track 35.3 -> 0.00 mm
- net /ACC_S0: track 34.8 -> 0.00 mm
- net /ALU_S2: track 33.7 -> 0.00 mm
- net /ALU_S3: track 32.2 -> 0.00 mm
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
Commit message: Register board
Parts:
- removed C1, C10, C11, C12, C13, C14, C15, C16, C2, C3, C4, C5, C6, C7, C8, C9: 100nF, Capacitor_SMD:C_0603_1608Metric_Pad1.08x0.95mm_HandSolder
- removed D10, D11, D12, D13, D14, D15, D16, D17, D18, D19, D2, D20, D21, D22, D23, D24, D25, D26, D27, D28, D29, D3, D30, D31, D32, D33, D34, D35, D4, D5, D6, D7, D8, D9: LED, LED_SMD:LED_0603_1608Metric_Pad1.05x0.95mm_HandSolder
- removed R10, R11, R12, R13, R17, R18, R19, R2, R20, R22, R23, R3, R36, R37, R38, R39, R4, R40, R41, R42, R43, R44, R45, R46, R47, R48, R49, R5, R50, R51, R6, R7, R8, R9: 330R, Resistor_SMD:R_0603_1608Metric_Pad0.98x0.95mm_HandSolder
- removed R14, R15, R16, R21, R24, R25, R26, R27, R28, R29, R30, R31, R32, R33, R34, R35, R52, R53, R54, R55, R56, R57, R58, R59, R60, R61, R62, R63, R64, R65, R66, R67, R68, R69, R70, R71, R72, R73, R74, R75, R76, R77, R78, R79, R80, R81, R82, R83, R84, R85, R86, R87, R88, R89, R90, R91, R92, R93, R94, R95, R96: 10K, Resistor_SMD:R_0603_1608Metric_Pad0.98x0.95mm_HandSolder
- added H1: MountingHole, MountingHole:MountingHole_3.5mm, F.Cu at (55.0, 48.2)
- added H2: MountingHole, MountingHole:MountingHole_3.5mm, F.Cu at (171.0, 48.2)
- added H3: MountingHole, MountingHole:MountingHole_3.5mm, F.Cu at (55.0, 123.2)
- added H4: MountingHole, MountingHole:MountingHole_3.5mm, F.Cu at (171.0, 123.2)
- added NT1: NetTie_2, NetTie:NetTie-2_SMD_Pad0.5mm, F.Cu at (144.1, 104.1)
- added RN1: R_Network08, Resistor_THT:R_Array_SIP9, F.Cu at (61.0, 70.5)
- added RN2: R_Network08, Resistor_THT:R_Array_SIP9, F.Cu at (61.0, 105.4)
- added RN3: R_Network08, Resistor_THT:R_Array_SIP9, F.Cu at (163.8, 110.5)
- added RN4: R_Network08, Resistor_THT:R_Array_SIP9, F.Cu at (163.8, 114.3)
- added U10: 74LS181, Package_DIP:DIP-24_W15.24mm_Socket, F.Cu at (125.7, 78.7)
- added U11: 74LS181, Package_DIP:DIP-24_W15.24mm_Socket, F.Cu at (148.6, 78.7)
- added U6: 74LS374, Package_DIP:DIP-20_W7.62mm_Socket, F.Cu at (121.9, 48.9)
- added U7: 74LS374, Package_DIP:DIP-20_W7.62mm_Socket, F.Cu at (133.3, 48.9)
- added U8: 74LS244, Package_DIP:DIP-20_W7.62mm_Socket, F.Cu at (144.8, 48.9)
- D1: footprint LED_SMD:LED_0603_1608Metric_Pad1.05x0.95mm_HandSolder -> LED_THT:LED_D3.0mm
- R1: footprint Resistor_SMD:R_0603_1608Metric_Pad0.98x0.95mm_HandSolder -> Resistor_THT:R_Axial_DIN0204_L3.6mm_D1.6mm_P2.54mm_Vertical
- moved J1 108.6 mm to (150.5, 120.0), turned to -90 degrees
- moved R1 84.0 mm to (159.4, 120.1), turned to -90 degrees
- moved D1 52.3 mm to (163.2, 122.6), turned to 90 degrees
- moved U13 42.0 mm to (76.2, 83.8)
- moved U12 42.0 mm to (64.8, 83.8)
- moved U14 42.0 mm to (87.6, 83.8)
- moved U15 42.0 mm to (99.1, 83.8)
- moved U16 42.0 mm to (110.5, 83.8)
- moved U3 39.1 mm to (87.6, 48.9)
- moved U1 39.1 mm to (64.8, 48.9)
- moved U2 39.1 mm to (76.2, 48.9)
- moved U4 39.1 mm to (99.1, 48.9)
- moved U5 39.1 mm to (110.5, 48.9)
- moved U9 10.0 mm to (156.2, 54.0)
- renumbered U2 to U12, U4 to U13, U6 to U14, U8 to U15, U10 to U16, U3 to U2, U5 to U3, U7 to U4, U9 to U5, U16 to U9
Connections:
- J1 pad 1: /A11 -> GND
- J1 pad 10: /A2 -> /D1
- J1 pad 11: /A1 -> /EQUAL_FLAG_A
- J1 pad 12: /A0 -> /CARRY_FLAG_A
- J1 pad 13: /A7 -> /FLAGS_B_UPDATE
- J1 pad 14: /A6 -> /FLAGS_A_UPDATE
- J1 pad 15: /A5 -> /EQUAL_FLAG_B
- J1 pad 16: /A4 -> /CARRY_FLAG_B
- J1 pad 17: /D3 -> /A_LOAD
- J1 pad 18: /D2 -> /T_LOAD
- J1 pad 19: /D1 -> /ALU_S2
- J1 pad 2: /A10 -> +5V
- J1 pad 20: /D0 -> /ALU_S3
- J1 pad 21: /D7 -> /ALU_S0
- J1 pad 22: /D6 -> /ALU_S1
- J1 pad 23: /D5 -> /D_LOAD
- J1 pad 24: /D4 -> /~{ALU_CIN}
- J1 pad 25: /~{PC_OUT} -> /~{ADR_L_OUT}
- J1 pad 26: /ALU_S0 -> /ALU_M
- J1 pad 27: /PC_H_LOAD -> /CLK
- J1 pad 28: /ALU_S1 -> /~{RESET}
- J1 pad 29: /PC_L_LOAD -> unconnected-(J1-Pin_29-Pad29)
- J1 pad 3: /A9 -> /D6
- J1 pad 30: /ALU_S2 -> /E_LOAD
- J1 pad 31: /~{SP_OUT} -> /C_LOAD
- J1 pad 32: /ALU_S3 -> /SP_L_LOAD
- J1 pad 33: /SP_H_LOAD -> /PC_L_LOAD
- J1 pad 34: /ALU_M -> /~{DE_OUT}
- J1 pad 35: /SP_L_LOAD -> /B_LOAD
- J1 pad 36: /~{ALU_CIN} -> /~{BC_OUT}
- J1 pad 37: /~{BC_OUT} -> /SP_H_LOAD
- J1 pad 38: /FLAGS_A_UPDATE -> /~{ADR_H_OUT}
- J1 pad 39: /B_LOAD -> /~{A_OUT}
- J1 pad 4: /A8 -> /D7
- J1 pad 40: /FLAGS_B_UPDATE -> /~{T_OUT}
- J1 pad 41: /C_LOAD -> /~{ALU_OUT}
- J1 pad 42: /CARRY_FLAG_A -> /~{PC_OUT}
- J1 pad 43: /~{DE_OUT} -> /PC_H_LOAD
- J1 pad 44: /EQUAL_FLAG_A -> /~{SP_OUT}
- J1 pad 45: /D_LOAD -> /A14
- J1 pad 46: /CARRY_FLAG_B -> /A13
- J1 pad 47: /E_LOAD -> /A12
- J1 pad 48: /EQUAL_FLAG_B -> /A15
- J1 pad 49: /~{ADR_H_OUT} -> /A4
- J1 pad 5: /A15 -> /D4
- J1 pad 50: /A_LOAD -> /A5
- J1 pad 51: /~{ADR_L_OUT} -> /A6
- J1 pad 52: /T_LOAD -> /A7
- J1 pad 53: /~{A_OUT} -> /A0
- J1 pad 54: /~{ALU_OUT} -> /A8
- J1 pad 55: /~{T_OUT} -> /A1
- J1 pad 56: unconnected-(J1-Pin_56-Pad56) -> /A9
- J1 pad 57: /~{RESET} -> /A2
- J1 pad 58: /CLK -> /A10
- J1 pad 59: GND -> /A3
- J1 pad 6: /A14 -> /D5
- J1 pad 60: +5V -> /A11
- J1 pad 7: /A13 -> /D2
- J1 pad 8: /A12 -> /D3
- J1 pad 9: /A3 -> /D0
Routing:
- net /ALU6: track 0.00 -> 273.2 mm, vias 0 -> 3
- net /ALU7: track 0.00 -> 267.9 mm, vias 0 -> 3
- net /ALU5: track 0.00 -> 257.0 mm, vias 0 -> 3
- net /ALU4: track 0.00 -> 247.6 mm, vias 0 -> 3
- net /ALU0: track 0.00 -> 237.6 mm, vias 0 -> 3
- net /ALU1: track 0.00 -> 229.3 mm, vias 0 -> 3
- net /ALU3: track 0.00 -> 226.3 mm, vias 0 -> 4
- net /ALU2: track 0.00 -> 215.0 mm, vias 0 -> 3
- net +5V: track 139.8 -> 344.3 mm, vias 0 -> 1
- net /~{ALU_OUT}: track 0.00 -> 163.8 mm
- net /L4: track 0.00 -> 155.5 mm, vias 0 -> 3
- net /L7: track 0.00 -> 151.9 mm, vias 0 -> 4
- net /L6: track 0.00 -> 151.2 mm, vias 0 -> 4
- net /L5: track 0.00 -> 148.4 mm, vias 0 -> 2
- net /~{T_OUT}: track 0.00 -> 145.5 mm
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Other:
- board outline added: 124 x 83 mm
- board text added: "A REG"
- board text added: "AH -> LEFT"
- board text added: "AL -> LEFT"
- board text added: "ALU -> DATA"
- board text added: "ALU HIGH"
- board text added: "ALU LOW"
- board text added: "B REG"
- board text added: "C REG"
- board text added: "D REG"
- board text added: "DATA MODULE"
- board text added: "E REG"
- board text added: "Ed Atkinson 2023"
- board text added: "FLAGS"
- board text added: "PC HIGH"
- board text added: "PC LOW"
- board text added: "POWER"
- board text added: "SP HIGH"
- board text added: "SP LOW"
- board text added: "T REG"

Commit message: Control panel schematic
Parts:
- removed D1: LED, LED_THT:LED_D3.0mm
- removed R1: 330R, Resistor_THT:R_Axial_DIN0204_L3.6mm_D1.6mm_P2.54mm_Vertical
- J1: value Conn_02x30_Odd_Even -> Conn_02x32_Odd_Even; footprint Connector_IDC:IDC-Header_2x30_P2.54mm_Vertical -> Connector_IDC:IDC-Header_2x32_P2.54mm_Vertical
- moved J1 2.54 mm to (153.0, 120.0)
Connections:
- J1 pad 29: unconnected-(J1-Pin_29-Pad29) -> /~{RAM_OUT}
- J1 pad 30: /E_LOAD -> /RAM_LOAD
- J1 pad 31: /C_LOAD -> unconnected-(J1-Pin_31-Pad31)
- J1 pad 32: /SP_L_LOAD -> unconnected-(J1-Pin_32-Pad32)
- J1 pad 33: /PC_L_LOAD -> /CONTROL_DISABLE
- J1 pad 34: /~{DE_OUT} -> /E_LOAD
- J1 pad 35: /B_LOAD -> /C_LOAD
- J1 pad 36: /~{BC_OUT} -> /SP_L_LOAD
- J1 pad 37: /SP_H_LOAD -> /PC_L_LOAD
- J1 pad 38: /~{ADR_H_OUT} -> /~{DE_OUT}
- J1 pad 39: /~{A_OUT} -> /B_LOAD
- J1 pad 40: /~{T_OUT} -> /~{BC_OUT}
- J1 pad 41: /~{ALU_OUT} -> /SP_H_LOAD
- J1 pad 42: /~{PC_OUT} -> /~{ADR_H_OUT}
- J1 pad 43: /PC_H_LOAD -> /~{A_OUT}
- J1 pad 44: /~{SP_OUT} -> /~{T_OUT}
- J1 pad 45: /A14 -> /~{ALU_OUT}
- J1 pad 46: /A13 -> /~{PC_OUT}
- J1 pad 47: /A12 -> /PC_H_LOAD
- J1 pad 48: /A15 -> /~{SP_OUT}
- J1 pad 49: /A4 -> /A14
- J1 pad 50: /A5 -> /A13
- J1 pad 51: /A6 -> /A12
- J1 pad 52: /A7 -> /A15
- J1 pad 53: /A0 -> /A4
- J1 pad 54: /A8 -> /A5
- J1 pad 55: /A1 -> /A6
- J1 pad 56: /A9 -> /A7
- J1 pad 57: /A2 -> /A0
- J1 pad 58: /A10 -> /A8
- J1 pad 59: /A3 -> /A1
- J1 pad 60: /A11 -> /A9
Routing:
- net Net-(D1-A): track 3.83 -> 0.00 mm
- net +5V: track 344.3 -> 340.6 mm
- net /A11: track 81.7 -> 78.5 mm
- net /D7: track 109.9 -> 107.3 mm
- net /A12: track 92.2 -> 89.7 mm
- net /EQUAL_FLAG_A: track 95.4 -> 92.9 mm
- net /A5: track 139.8 -> 137.3 mm
- net /~{PC_OUT}: track 141.6 -> 139.1 mm
- net /CARRY_FLAG_A: track 109.0 -> 106.4 mm
- net /A2: track 122.1 -> 119.6 mm
- net /A1: track 127.5 -> 125.0 mm
- net GND: track 1.80 -> 4.34 mm, vias 87 -> 94
- net /~{SP_OUT}: track 89.2 -> 86.6 mm
- net /FLAGS_B_UPDATE: track 97.2 -> 94.7 mm
- net /A9: track 101.0 -> 98.5 mm
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