File: Control_board/Control_board.kicad_sch (KiCad schematic)
At the start: 16 parts

Commit message: Control board progress
Parts:
- removed U? (x7): 74LS14, symbol 74xx:74LS14
- added J1 (x2): Conn_02x32_Odd_Even, Connector_IDC:IDC-Header_2x32_P2.54mm_Vertical, symbol Connector_Generic:Conn_02x32_Odd_Even
- added R1: 1K, Resistor_THT:R_Axial_DIN0204_L3.6mm_D1.6mm_P2.54mm_Vertical, symbol Device:R
- added RN1, RN2, RN3, RN4: R_Network08, Resistor_THT:R_Array_SIP9, symbol Device:R_Network08
- added U? (x3): 27C512, Package_DIP:DIP-28_W15.24mm, symbol Memory_EPROM:27C512
- NT?: footprint (none) -> NetTie:NetTie-2_SMD_Pad0.5mm
- U?: footprint (none) -> Package_DIP:DIP-16_W7.62mm_Socket
- U?: footprint (none) -> Package_DIP:DIP-20_W7.62mm_Socket
- U? (x2): footprint (none) -> Package_DIP:DIP-14_W7.62mm_Socket
Connections:
- net +5V: now also U?.28 (VCC), J1.2 (Pin_2), J1.2 (Pin_2), R1.1, RN2.1 (common), RN3.1 (common), U?.28 (VCC), U?.28 (VCC), U?.28 (VCC)
- net CLK: now also U?.22 (~{OE}), J1.27 (Pin_27), J1.27 (Pin_27), U?.22 (~{OE})
- net D0: now also J1.9 (Pin_9), J1.9 (Pin_9)
- net D1: now also J1.10 (Pin_10), J1.10 (Pin_10)
- net D2: now also J1.7 (Pin_7), J1.7 (Pin_7)
- net D3: now also J1.8 (Pin_8), J1.8 (Pin_8)
- net D4: now also J1.5 (Pin_5), J1.5 (Pin_5)
- net D5: now also J1.6 (Pin_6), J1.6 (Pin_6)
- net D6: now also J1.3 (Pin_3), J1.3 (Pin_3)
- net D7: now also J1.4 (Pin_4), J1.4 (Pin_4)
- net GND: now also U?.14 (GND), J1.1 (Pin_1), J1.1 (Pin_1), RN1.1 (common), RN4.1 (common), U?.14 (GND), U?.14 (GND), U?.14 (GND), U?.22 (~{OE}), U?.22 (~{OE}); no longer U?.14 (CLR)
- net MA0: now also U?.10 (A0), U?.10 (A0), U?.10 (A0)
- net MA1: now also U?.9 (A1), U?.9 (A1), U?.9 (A1)
- net MA10: now also U?.21 (A10), U?.21 (A10), U?.21 (A10)
- net MA11: now also U?.23 (A11), U?.23 (A11), U?.23 (A11)
- net MA12: now also U?.2 (A12), U?.2 (A12), U?.2 (A12)
- net MA13: now also U?.26 (A13), U?.26 (A13), U?.26 (A13)
- net MA14: now also U?.27 (A14), U?.27 (A14), U?.27 (A14)
- net MA15: now also U?.1 (A15), U?.1 (A15), U?.1 (A15)
- net MA2: now also U?.8 (A2), U?.8 (A2), U?.8 (A2)
- net MA3: now also U?.7 (A3), U?.7 (A3), U?.7 (A3)
- net MA4: now also U?.6 (A4), U?.6 (A4), U?.6 (A4)
- net MA5: now also U?.5 (A5), U?.5 (A5), U?.5 (A5)
- net MA6: now also U?.4 (A6), U?.4 (A6), U?.4 (A6)
- net MA7: now also U?.3 (A7), U?.3 (A7), U?.3 (A7)
- net MA8: now also U?.25 (A8), U?.25 (A8), U?.25 (A8)
- net MA9: now also U?.24 (A9), U?.24 (A9), U?.24 (A9)
- net ~{RESET}: now also J1.28 (Pin_28), J1.28 (Pin_28)
- net PC_H_LOAD: now reaches U?.11 (D0)
- net PC_H_LOAD: now also J1.47 (Pin_47), J1.47 (Pin_47), RN1.2 (R1)
- net PC_L_LOAD: now reaches U?.12 (D1)
- net PC_L_LOAD: now also J1.37 (Pin_37), J1.37 (Pin_37), RN1.3 (R2)
- net SP_H_LOAD: now reaches U?.13 (D2)
- net SP_H_LOAD: now also J1.41 (Pin_41), J1.41 (Pin_41), RN1.4 (R3)
- net SP_L_LOAD: now reaches U?.15 (D3)
- net SP_L_LOAD: now also J1.36 (Pin_36), J1.36 (Pin_36), RN1.5 (R4)
- net B_LOAD: now reaches U?.16 (D4)
- net B_LOAD: now also J1.39 (Pin_39), J1.39 (Pin_39), RN1.6 (R5)
- net C_LOAD: now reaches U?.17 (D5)
- net C_LOAD: now also J1.35 (Pin_35), J1.35 (Pin_35), RN1.7 (R6)
- net D_LOAD: now reaches U?.18 (D6)
- net D_LOAD: now also J1.23 (Pin_23), J1.23 (Pin_23), RN1.8 (R7)
- net E_LOAD: now reaches U?.19 (D7)
- net E_LOAD: now also J1.34 (Pin_34), J1.34 (Pin_34), RN1.9 (R8)
- net CONTROL_DISABLE: now reaches U?.20 (~{CE})
- net CONTROL_DISABLE: now also J1.33 (Pin_33), J1.33 (Pin_33), U?.20 (~{CE}), U?.20 (~{CE}), U?.20 (~{CE})
- net FLAGS_A_CARRY renamed CARRY_FLAG_A
- net CARRY_FLAG_A: now also J1.12 (Pin_12), J1.12 (Pin_12)
- net FLAGS_A_EQUAL renamed EQUAL_FLAG_A
- net EQUAL_FLAG_A: now also J1.11 (Pin_11), J1.11 (Pin_11)
- net FLAGS_B_CARRY renamed CARRY_FLAG_B
- net CARRY_FLAG_B: now also J1.16 (Pin_16), J1.16 (Pin_16)
- net FLAG_INTERRUPT renamed INTERRUPT_FLAG
- net INTERRUPT_FLAG: now also J1.31 (Pin_31), J1.31 (Pin_31)
- new net A0: J1.57 (Pin_57), J1.57 (Pin_57)
- new net A1: J1.59 (Pin_59), J1.59 (Pin_59)
- new net A10: J1.62 (Pin_62), J1.62 (Pin_62)
- new net A11: J1.64 (Pin_64), J1.64 (Pin_64)
- new net A12: J1.51 (Pin_51), J1.51 (Pin_51)
- new net A13: J1.50 (Pin_50), J1.50 (Pin_50)
- new net A14: J1.49 (Pin_49), J1.49 (Pin_49)
- new net A15: J1.52 (Pin_52), J1.52 (Pin_52)
- new net A2: J1.61 (Pin_61), J1.61 (Pin_61)
- new net A3: J1.63 (Pin_63), J1.63 (Pin_63)
- new net A4: J1.53 (Pin_53), J1.53 (Pin_53)
- new net A5: J1.54 (Pin_54), J1.54 (Pin_54)
- new net A6: J1.55 (Pin_55), J1.55 (Pin_55)
- new net A7: J1.56 (Pin_56), J1.56 (Pin_56)
- new net A8: J1.58 (Pin_58), J1.58 (Pin_58)
- new net A9: J1.60 (Pin_60), J1.60 (Pin_60)
- new net ALU_M: J1.26 (Pin_26), J1.26 (Pin_26), RN2.7 (R6), U?.13 (D2)
- new net ALU_S0: J1.21 (Pin_21), J1.21 (Pin_21), RN2.6 (R5), U?.15 (D3)
- new net ALU_S1: J1.22 (Pin_22), J1.22 (Pin_22), RN2.5 (R4), U?.16 (D4)
- new net ALU_S2: J1.19 (Pin_19), J1.19 (Pin_19), RN2.4 (R3), U?.17 (D5)
- new net ALU_S3: J1.20 (Pin_20), J1.20 (Pin_20), RN2.3 (R2), U?.18 (D6)
- new net A_LOAD: J1.17 (Pin_17), J1.17 (Pin_17), RN4.2 (R1), U?.11 (D0)
- new net COUNTER_RESET: RN4.7 (R6), U?.14 (CLR), U?.17 (D5)
- new net EQUAL_FLAG_B: J1.15 (Pin_15), J1.15 (Pin_15)
- new net FLAGS_A_UPDATE: J1.14 (Pin_14), J1.14 (Pin_14), RN4.8 (R7), U?.18 (D6)
- new net FLAGS_B_UPDATE: J1.13 (Pin_13), J1.13 (Pin_13), RN4.9 (R8), U?.19 (D7)
- new net T_LOAD: J1.18 (Pin_18), J1.18 (Pin_18), RN4.3 (R2), U?.12 (D1)
- new net ~{ADR_H_OUT}: J1.42 (Pin_42), J1.42 (Pin_42), RN2.8 (R7), U?.12 (D1)
- new net ~{ADR_L_OUT}: J1.25 (Pin_25), J1.25 (Pin_25), RN2.9 (R8), U?.11 (D0)
- new net ~{ALU_CIN}: J1.24 (Pin_24), J1.24 (Pin_24), RN2.2 (R1), U?.19 (D7)
- new net ~{ALU_OUT}: J1.45 (Pin_45), J1.45 (Pin_45), RN3.3 (R2), U?.18 (D6)
- new net ~{A_OUT}: J1.43 (Pin_43), J1.43 (Pin_43), RN3.5 (R4), U?.16 (D4)
- new net ~{BC_OUT}: J1.40 (Pin_40), J1.40 (Pin_40), RN3.7 (R6), U?.13 (D2)
- new net ~{DE_OUT}: J1.38 (Pin_38), J1.38 (Pin_38), RN3.6 (R5), U?.15 (D3)
- new net ~{PC_OUT}: J1.46 (Pin_46), J1.46 (Pin_46), RN3.9 (R8), U?.11 (D0)
- new net ~{RAM_LOAD}: J1.30 (Pin_30), J1.30 (Pin_30), R1.2, U?.13 (D2)
- new net ~{RAM_OUT}: J1.29 (Pin_29), J1.29 (Pin_29), RN3.2 (R1), U?.19 (D7)
- new net ~{SP_OUT}: J1.48 (Pin_48), J1.48 (Pin_48), RN3.8 (R7), U?.12 (D1)
- new net ~{T_OUT}: J1.44 (Pin_44), J1.44 (Pin_44), RN3.4 (R3), U?.17 (D5)
- no-connect marks 2 -> 9
Other:
- note added: "Connect clock to microcode rom ~{OE} selected write lines will fire on low clock"
- note added: "Could add two decoders to save an EEPROM Not really worth it though imo"
- note added: "Do I need a clear interrupt signal?"
- note added: "Interrupt will need to be latched and not change mid instruction"
- note added: "TODO clock generator"
- note added: "~{RESET} will load opcode 0x00 to IR and reset counter This will then load a predefined value tbd to PC"
- note removed: "4x microcode roms"
- note removed: "All microcode ~{CE} will be connect to a pin on the module connector This will allow a debug display module to take over and pull all the register contents"
- note removed: "TODO Clock generator Will also need an inverted clock"
- note removed: "Will invert the clock and use it on microcode rom ~{OE} for timing the register load signals"
- note removed: "Will need to latch interrupt on the IO board"
- moved on the sheet: U?, U?A, U?B

Commit message: No progress but more thoughts
Parts:
- removed U? (x2): LM556, Package_DIP:DIP-14_W7.62mm_Socket, symbol Timer:LM556
- added RV1: R_Potentiometer, symbol Device:R_Potentiometer
- added SW1: SW_Push, symbol Switch:SW_Push
- added U1: 74LS373, symbol 74xx:74LS373
- added U2: ATtiny85-20P, Package_DIP:DIP-8_W7.62mm_Socket, symbol MCU_Microchip_ATtiny:ATtiny85-20P
- added U4: 74LS123, Package_DIP:DIP-16_W7.62mm_Socket, symbol 74xx:74LS123
Connections:
- net HALT: now reaches U?.16 (D4)
- net HALT: now also RN4.6 (R5)
- no-connect marks 9 -> 7
Other:
- note added: "EEPROM address changes on clock rising edge Control lines settle during clock high Writes occur on clock falling edge"
- note added: "This is where using a latch for flags has come back to haunt me Update line needs to be high during clock high but only if wanted But also flags changing could cause a feedback loop aaahhhhhhhh Gonna have to add a monostable trigger, so didn't end up saving a chip lol Could also bypass the latch and add new flip-flops on this board Then would make sense to add one for interrupt flag too"

Commit message: Clock generator done... probably
Parts:
- added D1, D2: LED, LED_THT:LED_D2.0mm_W4.8mm_H2.5mm_FlatTop, symbol Device:LED
- added J3: ICSP, Connector_PinHeader_2.54mm:PinHeader_2x03_P2.54mm_Vertical, symbol Connector_Generic:Conn_02x03_Odd_Even
- added R2, R3: 330R, Resistor_THT:R_Axial_DIN0204_L3.6mm_D1.6mm_P2.54mm_Vertical, symbol Device:R
- added SW2: SW_Push, symbol Switch:SW_Push
Connections:
- net +5V: now also RV1.3, U2.8 (VCC), J3.2 (Pin_2)
- net CLK: now also U2.3 (XTAL2/PB4), D1.2 (A)
- net GND: now also RV1.1, SW1.2, U2.4 (GND), J3.6 (Pin_6), R2.2, R3.2, SW2.2
- net at SW1.1: now also U2.5 (AREF/PB0), J3.4 (Pin_4)
- net at RV1.2: now also U2.2 (XTAL1/PB3)
- net at U2.1 (~{RESET}/PB5): now also J3.5 (Pin_5)
- net at U2.6 (PB1): now also D2.2 (A), J3.1 (Pin_1)
- net at U2.7 (PB2): now also J3.3 (Pin_3), SW2.1
- new net: D1.1 (K), R2.1
- new net: D2.1 (K), R3.1
Other:
- note added: "Clock LED"
- note added: "Is an attiny cheating, its only doing what could be done with a 555 But this gives me flexibility for trying different clock speeds and can debounce the single step button for me This project is about TTL logic not the 555 lol"
- note added: "Mode LED"
- note added: "Mode button"
- note added: "Single step button"
- note removed: "TODO clock generator"
- moved on the sheet: RV1, SW1

Commit message: Control board schematic done?
Parts:
- removed NT? (x4): NetTie_2, NetTie:NetTie-2_SMD_Pad0.5mm, symbol Device:NetTie_2
- removed U4: 74LS123, Package_DIP:DIP-16_W7.62mm_Socket, symbol 74xx:74LS123
- added U1, U2: 74LS74, Package_DIP:DIP-14_W7.62mm_Socket, symbol 74xx:74LS74
- added U4: 74LS373, Package_DIP:DIP-20_W7.62mm_Socket, symbol 74xx:74LS373
- R1: footprint Resistor_THT:R_Axial_DIN0204_L3.6mm_D1.6mm_P2.54mm_Vertical -> Resistor_THT:R_Axial_DIN0207_L6.3mm_D2.5mm_P7.62mm_Horizontal
- R2: renamed from R3; footprint Resistor_THT:R_Axial_DIN0204_L3.6mm_D1.6mm_P2.54mm_Vertical -> Resistor_THT:R_Axial_DIN0207_L6.3mm_D2.5mm_P7.62mm_Horizontal
- R3: renamed from R2; footprint Resistor_THT:R_Axial_DIN0204_L3.6mm_D1.6mm_P2.54mm_Vertical -> Resistor_THT:R_Axial_DIN0207_L6.3mm_D2.5mm_P7.62mm_Horizontal
- RV1: footprint (none) -> Potentiometer_THT:Potentiometer_Bourns_3386F_Vertical
- SW1: renamed from SW2; footprint (none) -> Button_Switch_THT:SW_PUSH_6mm
- SW2: renamed from SW1; footprint (none) -> Button_Switch_THT:SW_PUSH_6mm
- U10, U7, U8, U9: renamed from U?; footprint Package_DIP:DIP-28_W15.24mm -> Package_DIP:DIP-28_W15.24mm_Socket
- U6: renamed from U1; footprint (none) -> Package_DIP:DIP-20_W7.62mm_Socket
- gave numbers to parts that had none: 2
- renumbered D2 to D1, D1 to D2, J3 to J1, RN4 to RN1, RN1 to RN2, RN2 to RN4, U2 to U11
Connections:
- net +5V: now also U6.20 (VCC), U1.14 (VCC), U2.14 (VCC), U4.20 (VCC)
- net CLK: now also U6.11 (LE), U4.11 (LE)
- net COUNTER_RESET: now also RN1.6 (R5), U8.16 (D4); no longer RN1.7 (R6), U8.17 (D5)
- net FLAGS_A_UPDATE: now also U1.11 (C), U1.3 (C); no longer J1.14 (Pin_14), J1.14 (Pin_14)
- net FLAGS_B_UPDATE: now also U2.3 (C); no longer J1.13 (Pin_13), J1.13 (Pin_13)
- net GND: now also U6.1 (OE), U6.10 (GND), U1.7 (GND), U2.7 (GND), U4.1 (OE), U4.10 (GND), U4.13 (D4), U4.14 (D5), U4.17 (D6), U4.18 (D7)
- net HALT: no longer RN1.6 (R5), U8.16 (D4)
- net INTERRUPT_FLAG: now also J1.13 (Pin_13), J1.13 (Pin_13), U2.12 (D); no longer J1.31 (Pin_31), J1.31 (Pin_31)
- net MA10: now also U6.16 (O6); no longer U3.16 (Q6)
- net MA11: now also U6.19 (O7); no longer U3.19 (Q7)
- net MA12: now also U4.2 (O0)
- net MA13: now also U4.5 (O1)
- net MA14: now also U4.6 (O2)
- net MA15: now also U4.9 (O3)
- net MA4: now also U6.2 (O0); no longer U3.2 (Q0)
- net MA5: now also U6.5 (O1); no longer U3.5 (Q1)
- net MA6: now also U6.6 (O2); no longer U3.6 (Q2)
- net MA7: now also U6.9 (O3); no longer U3.9 (Q3)
- net MA8: now also U6.12 (O4); no longer U3.12 (Q4)
- net MA9: now also U6.15 (O5); no longer U3.15 (Q5)
- net ~{RESET}: now also U2.13 (~{R})
- net at U6.13 (D4): now also U3.12 (Q4)
- net at U6.14 (D5): now also U3.15 (Q5)
- net at U6.17 (D6): now also U3.16 (Q6)
- net at U6.18 (D7): now also U3.19 (Q7)
- net at U6.3 (D0): now also U3.2 (Q0)
- net at U6.4 (D1): now also U3.5 (Q1)
- net at U6.7 (D2): now also U3.6 (Q2)
- net at U6.8 (D3): now also U3.9 (Q3)
- net CARRY_FLAG_A renamed CARRY_FLAG
- net CARRY_FLAG: now also U1.2 (D), U2.2 (D)
- net CARRY_FLAG_B: no longer names the net of J1.16 (Pin_16)
- net CARRY_FLAG_B: no longer J1.16 (Pin_16)
- net EQUAL_FLAG_A renamed EQUAL_FLAG
- net EQUAL_FLAG: now also U1.12 (D)
- net EQUAL_FLAG_B: no longer names the net of J1.15 (Pin_15)
- net EQUAL_FLAG_B: no longer J1.15 (Pin_15)
- new net: U2.5 (Q), U4.7 (D2)
- new net: U2.9 (Q), U4.8 (D3)
- new net: U1.5 (Q), U4.3 (D0)
- new net: U1.9 (Q), U4.4 (D1)
- new net INTERRUPT_UPDATE: RN1.7 (R6), U2.11 (C), U8.17 (D5)
- no-connect marks 7 -> 30
Other:
- note added: "Flags updated on falling edge clock then latch delays change until high clock"
- note added: "IR loads on falling edge clock then latch delays change until high clock"
- note removed: "Interrupt will need to be latched and not change mid instruction"
- note removed: "This is where using a latch for flags has come back to haunt me Update line needs to be high during clock high but only if wanted But also flags changing could cause a feedback loop aaahhhhhhhh Gonna have to add a monostable trigger, so didn't end up saving a chip lol Could also bypass the latch and add new flip-flops on this board Then would make sense to add one for interrupt flag too"
- moved on the sheet: D1, D2, J1, R1, R2, R3, RN1, RN2, RN3, RN4, RV1, SW1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

Commit message: Control board ready for routing
Parts:
- added D10, D11, D12, D13, D14, D15, D16, D17, D18, D19, D20, D21, D22, D23, D24, D25, D26, D27, D28, D29, D3, D30, D31, D32, D33, D34, D35, D36, D37, D38, D39, D4, D40, D41, D42, D43, D44, D45, D46, D47, D48, D49, D5, D50, D51, D52, D6, D7, D8, D9: LED, LED_THT:LED_D2.0mm_W4.8mm_H2.5mm_FlatTop, symbol Device:LED
- added H1, H2, H3, H4: MountingHole, MountingHole:MountingHole_3.5mm, symbol Mechanical:MountingHole
- added R10, R11, R13, R5, R6: 1K, Resistor_THT:R_Axial_DIN0207_L6.3mm_D2.5mm_P7.62mm_Horizontal, symbol Device:R
- added R12, R4, R7, R8, R9: 330R, Resistor_THT:R_Axial_DIN0207_L6.3mm_D2.5mm_P7.62mm_Horizontal, symbol Device:R
- added RN10, RN5, RN6, RN7, RN8, RN9: 330R, Resistor_THT:R_Array_SIP9, symbol Device:R_Network08
- added SW3, SW4: SW_Push, Button_Switch_THT:SW_PUSH_6mm, symbol Switch:SW_Push
- added U12: 74LS74, Package_DIP:DIP-14_W7.62mm_Socket, symbol 74xx:74LS74
- RN1, RN2, RN3, RN4: value R_Network08 -> 1K
Connections:
- net +5V: now also U1.1 (~{R}), U1.10 (~{S}), U1.13 (~{R}), U1.4 (~{S}), U2.1 (~{R}), U2.10 (~{S}), U2.13 (~{R}), U2.4 (~{S}), R10.1, R13.1, R5.1, R6.1, R7.2, R8.2, R9.2, RN10.1 (common), RN9.1 (common), U12.14 (VCC), U12.4 (~{S})
- net ALU_M: now also D46.1 (K)
- net ALU_S0: now also D47.1 (K)
- net ALU_S1: now also D48.1 (K)
- net ALU_S2: now also D49.1 (K)
- net ALU_S3: now also D50.1 (K)
- net A_LOAD: now also D23.2 (A)
- net B_LOAD: now also D32.2 (A)
- net CONTROL_DISABLE: now also D52.2 (A), R11.1
- net COUNTER_RESET: now also RN1.5 (R4), U8.15 (D3), D25.2 (A), U12.3 (C); no longer RN1.6 (R5), U8.16 (D4)
- net C_LOAD: now also D33.2 (A)
- net D_LOAD: now also D34.2 (A)
- net E_LOAD: now also D35.2 (A)
- net FLAGS_A_UPDATE: now also D26.2 (A)
- net FLAGS_B_UPDATE: now also D27.2 (A)
- net GND: now also U2.11 (C), U2.12 (D), R11.2, R12.2, R4.2, RN5.1 (common), RN6.1 (common), RN7.1 (common), RN8.1 (common), SW3.2, SW4.2, U12.11 (C), U12.12 (D), U12.7 (GND); no longer U4.13 (D4), U4.14 (D5), U4.17 (D6), U4.18 (D7)
- net MA0: now also U4.2 (O0), D3.2 (A); no longer U5.3 (QA)
- net MA1: now also U4.5 (O1), D4.2 (A); no longer U5.2 (QB)
- net MA10: now also U6.6 (O2), D14.2 (A); no longer U6.16 (O6)
- net MA11: now also U6.9 (O3), D15.2 (A); no longer U6.19 (O7)
- net MA12: now also U6.12 (O4), D16.2 (A); no longer U4.2 (O0)
- net MA13: now also U6.15 (O5), D17.2 (A); no longer U4.5 (O1)
- net MA14: now also U6.16 (O6), D18.2 (A); no longer U4.6 (O2)
- net MA15: now also U6.19 (O7), D19.2 (A); no longer U4.9 (O3)
- net MA2: now also U4.6 (O2), D5.2 (A); no longer U5.6 (QC)
- net MA3: now also U4.9 (O3), D7.2 (A); no longer U5.7 (QD)
- net MA4: now also U4.12 (O4), D8.2 (A); no longer U6.2 (O0)
- net MA5: now also U4.15 (O5), D9.2 (A); no longer U6.5 (O1)
- net MA6: now also U4.16 (O6), D10.2 (A); no longer U6.6 (O2)
- net MA7: now also U4.19 (O7), D11.2 (A); no longer U6.9 (O3)
- net MA8: now also U6.2 (O0), D12.2 (A); no longer U6.12 (O4)
- net MA9: now also U6.5 (O1), D13.2 (A); no longer U6.15 (O5)
- net PC_H_LOAD: now also D28.2 (A)
- net PC_L_LOAD: now also D29.2 (A)
- net SP_H_LOAD: now also D30.2 (A)
- net SP_L_LOAD: now also D31.2 (A)
- net T_LOAD: now also D24.2 (A)
- net ~{ADR_H_OUT}: now also D45.1 (K)
- net ~{ADR_L_OUT}: now also D44.1 (K)
- net ~{ALU_CIN}: now also D51.1 (K)
- net ~{ALU_OUT}: now also D42.1 (K)
- net ~{A_OUT}: now also D40.1 (K)
- net ~{BC_OUT}: now also D38.1 (K)
- net ~{DE_OUT}: now also D39.1 (K)
- net ~{PC_OUT}: now also D36.1 (K)
- net ~{RAM_LOAD}: now also D22.1 (K)
- net ~{RAM_OUT}: now also D43.1 (K)
- net ~{RESET}: now also R10.2, SW3.1; no longer U2.13 (~{R})
- net ~{SP_OUT}: now also D37.1 (K)
- net ~{T_OUT}: now also D41.1 (K)
- net at U2.5 (Q): now also U4.17 (D6); no longer U4.7 (D2)
- net at U4.8 (D3): now also U5.7 (QD); no longer U2.9 (Q)
- net at U4.3 (D0): now also U5.3 (QA); no longer U1.5 (Q)
- net at U4.4 (D1): now also U5.2 (QB); no longer U1.9 (Q)
- net INTERRUPT_FLAG renamed ~{INTERRUPT_FLAG}
- net ~{INTERRUPT_FLAG}: now also R13.2, SW4.1, U12.2 (D); no longer U2.12 (D)
- removed net INTERRUPT_UPDATE: RN1.7 (R6), U2.11 (C), U8.17 (D5)
- new net: D25.1 (K), RN7.5 (R4)
- new net: D3.1 (K), RN5.9 (R8)
- new net: D19.1 (K), RN6.2 (R1)
- new net: D43.2 (A), RN9.2 (R1)
- new net: D15.1 (K), RN6.6 (R5)
- new net: D18.1 (K), RN6.3 (R2)
- new net: D28.1 (K), RN8.2 (R1)
- new net: D6.1 (K), R4.1
- new net: D6.2 (A), U12.1 (~{R}), U12.9 (Q)
- new net: D34.1 (K), RN8.8 (R7)
- new net: D32.1 (K), RN8.6 (R5)
- new net: D45.2 (A), RN10.8 (R7)
- new net: D14.1 (K), RN6.7 (R6)
- new net: D17.1 (K), RN6.4 (R3)
- new net: D31.1 (K), RN8.5 (R4)
- new net: D29.1 (K), RN8.3 (R2)
- new net: D36.2 (A), RN9.9 (R8)
- new net: D20.2 (A), R7.1
- new net: D27.1 (K), RN7.9 (R8)
- new net: D21.2 (A), R8.1
- new net: U4.7 (D2), U5.6 (QC)
- new net: D30.1 (K), RN8.4 (R3)
- new net: D40.2 (A), RN9.5 (R4)
- new net: D41.2 (A), RN9.4 (R3)
- new net: D10.1 (K), RN5.3 (R2)
- new net: D33.1 (K), RN8.7 (R6)
- new net: D35.1 (K), RN8.9 (R8)
- new net: D38.2 (A), RN9.7 (R6)
- new net: D22.2 (A), R9.1
- new net: D47.2 (A), RN10.6 (R5)
- new net: D7.1 (K), RN5.6 (R5)
- new net: D42.2 (A), RN9.3 (R2)
- new net: D39.2 (A), RN9.6 (R5)
- new net: D37.2 (A), RN9.8 (R7)
- new net: D9.1 (K), RN5.4 (R3)
- new net: D50.2 (A), RN10.3 (R2)
- new net: D48.2 (A), RN10.5 (R4)
- new net: D12.1 (K), RN6.9 (R8)
- new net: D8.1 (K), RN5.5 (R4)
- new net: D24.1 (K), RN7.3 (R2)
- new net: D46.2 (A), RN10.7 (R6)
- new net: D23.1 (K), RN7.2 (R1)
- new net: D5.1 (K), RN5.7 (R6)
- new net: D52.1 (K), R12.1
- new net: D16.1 (K), RN6.5 (R4)
- new net: D13.1 (K), RN6.8 (R7)
- new net: U1.5 (Q), U4.13 (D4)
- new net: D11.1 (K), RN5.2 (R1)
- new net: D49.2 (A), RN10.4 (R3)
- new net: D26.1 (K), RN7.8 (R7)
- new net: U12.5 (Q), U4.18 (D7)
- new net: U1.9 (Q), U4.14 (D5)
- new net: D4.1 (K), RN5.8 (R7)
- new net: D51.2 (A), RN10.2 (R1)
- new net: D44.2 (A), RN10.9 (R8)
- new net ~{INTERRUPT_DISABLE}: D20.1 (K), R5.2, U12.10 (~{S}), U8.17 (D5)
- new net ~{INTERRUPT_ENABLE}: D21.1 (K), R6.2, U12.13 (~{R}), U8.16 (D4)
- no-connect marks 30 -> 25
Other:
- note added: "Count occurs on rising edge clock, latch is only nescessary for the asynchronous resets"
- note added: "Flags updated on falling edge clock then latch delays change until high clock Interrupt updates on rising edge clock, can be held in reset to disable interrupts"
- note removed: "Do I need a clear interrupt signal?"
- note removed: "Flags updated on falling edge clock then latch delays change until high clock"
- moved on the sheet: U1A, U1B, U1C, U2A, U2B, U2C, U4, U5

Commit message: Control board and connector bridge ready for ordering
Parts:
- removed J1: Conn_02x32_Odd_Even, Connector_IDC:IDC-Header_2x32_P2.54mm_Vertical, symbol Connector_Generic:Conn_02x32_Odd_Even
- added J3: Conn_01x02, Connector_PinHeader_2.54mm:PinHeader_1x02_P2.54mm_Vertical, symbol Connector_Generic:Conn_01x02
- renumbered D36 to D28, D37 to D29, D38 to D30, D39 to D31, D40 to D32, D41 to D33, D42 to D34, D43 to D35, D28 to D36, D29 to D37, D30 to D38, D31 to D39, D32 to D40, D33 to D41, D34 to D42, D35 to D43, R5 to R1, R6 to R5, R1 to R6, RN9 to RN8, RN8 to RN9, U8 to U10, U9 to U7, U7 to U8, U10 to U9
Connections:
- net +5V: now also U12.10 (~{S}), J3.2 (Pin_2)
- net ALU_M: now also D45.1 (K), RN4.3 (R2), U9.12 (D1); no longer D46.1 (K), RN4.7 (R6), U9.13 (D2)
- net ALU_S0: now also D48.1 (K), U9.16 (D4); no longer D47.1 (K), U9.15 (D3)
- net ALU_S1: now also D49.1 (K), RN4.7 (R6), U9.17 (D5); no longer D48.1 (K), RN4.5 (R4), U9.16 (D4)
- net ALU_S2: now also D50.1 (K), RN4.8 (R7), U9.18 (D6); no longer D49.1 (K), RN4.4 (R3), U9.17 (D5)
- net ALU_S3: now also D51.1 (K), RN4.9 (R8), U9.19 (D7); no longer D50.1 (K), RN4.3 (R2), U9.18 (D6)
- net B_LOAD: now also D38.2 (A), RN2.4 (R3), U8.13 (D2); no longer D40.2 (A), RN2.6 (R5), U8.16 (D4)
- net C_LOAD: now also D40.2 (A), RN2.6 (R5), U8.16 (D4); no longer D41.2 (A), RN2.7 (R6), U8.17 (D5)
- net D_LOAD: now also D43.2 (A), RN2.9 (R8), U8.19 (D7); no longer D42.2 (A), RN2.8 (R7), U8.18 (D6)
- net E_LOAD: now also D42.2 (A), RN2.8 (R7), U8.18 (D6); no longer D43.2 (A), RN2.9 (R8), U8.19 (D7)
- net GND: now also J3.1 (Pin_1); no longer U12.11 (C), U12.12 (D)
- net IR_LOAD: now also D20.1 (K), R1.2, U10.17 (D5)
- net PC_L_LOAD: now also D39.2 (A), RN2.5 (R4), U8.15 (D3); no longer D37.2 (A), RN2.3 (R2), U8.12 (D1)
- net SP_H_LOAD: now also D37.2 (A), RN2.3 (R2), U8.12 (D1); no longer D38.2 (A), RN2.4 (R3), U8.13 (D2)
- net SP_L_LOAD: now also D41.2 (A), RN2.7 (R6), U8.17 (D5); no longer D39.2 (A), RN2.5 (R4), U8.15 (D3)
- net ~{ADR_H_OUT}: now also D44.1 (K), RN4.2 (R1), U9.11 (D0); no longer D45.1 (K), RN4.8 (R7), U9.12 (D1)
- net ~{ADR_L_OUT}: now also D46.1 (K), RN4.4 (R3), U9.13 (D2); no longer D44.1 (K), RN4.9 (R8), U9.11 (D0)
- net ~{ALU_CIN}: now also D47.1 (K), RN4.5 (R4), U9.15 (D3); no longer D51.1 (K), RN4.2 (R1), U9.19 (D7)
- net ~{ALU_OUT}: now also D29.1 (K), U7.12 (D1); no longer D34.1 (K), U7.18 (D6)
- net ~{A_OUT}: now also D31.1 (K), U7.15 (D3); no longer D32.1 (K), U7.16 (D4)
- net ~{BC_OUT}: now also D33.1 (K), U7.17 (D5); no longer D30.1 (K), U7.13 (D2)
- net ~{DE_OUT}: now also D34.1 (K), RN3.8 (R7), U7.18 (D6); no longer D31.1 (K), RN3.6 (R5), U7.15 (D3)
- net ~{PC_OUT}: now also D30.1 (K), RN3.4 (R3), U7.13 (D2); no longer D28.1 (K), RN3.9 (R8), U7.11 (D0)
- net ~{RAM_OUT}: now also RN3.9 (R8); no longer RN3.2 (R1)
- net ~{RESET}: now also U12.13 (~{R})
- net ~{SP_OUT}: now also D28.1 (K), RN3.2 (R1), U7.11 (D0); no longer D29.1 (K), RN3.8 (R7), U7.12 (D1)
- net ~{T_OUT}: now also D32.1 (K), RN3.6 (R5), U7.16 (D4); no longer D33.1 (K), RN3.4 (R3), U7.17 (D5)
- net at D35.2 (A): now also RN8.9 (R8); no longer RN8.2 (R1)
- net at D45.2 (A): now also RN10.3 (R2); no longer RN10.8 (R7)
- net at D28.2 (A): now also RN8.2 (R1); no longer RN8.9 (R8)
- net at D32.2 (A): now also RN8.6 (R5); no longer RN8.5 (R4)
- net at D33.2 (A): now also RN8.7 (R6); no longer RN8.4 (R3)
- net at D30.2 (A): now also RN8.4 (R3); no longer RN8.7 (R6)
- net at D47.2 (A): now also RN10.5 (R4); no longer RN10.6 (R5)
- net at RN8.3 (R2): now also D29.2 (A); no longer D34.2 (A)
- net at D31.2 (A): now also RN8.5 (R4); no longer RN8.6 (R5)
- net at RN8.8 (R7): now also D34.2 (A); no longer D29.2 (A)
- net at D50.2 (A): now also RN10.8 (R7); no longer RN10.3 (R2)
- net at D48.2 (A): now also RN10.6 (R5); no longer RN10.5 (R4)
- net at D46.2 (A): now also RN10.4 (R3); no longer RN10.7 (R6)
- net at D49.2 (A): now also RN10.7 (R6); no longer RN10.4 (R3)
- net at U12.8 (~{Q}): now also U12.12 (D)
- net at D51.2 (A): now also RN10.9 (R8); no longer RN10.2 (R1)
- net at D44.2 (A): now also RN10.2 (R1); no longer RN10.9 (R8)
- removed net ~{INTERRUPT_DISABLE}: D20.1 (K), R1.2, U10.17 (D5), U12.10 (~{S})
- net ~{INTERRUPT_ENABLE} renamed INT_EN_TOGGLE
- net INT_EN_TOGGLE: now also U12.11 (C); no longer U12.13 (~{R})
- no-connect marks 25 -> 35
Other:
- moved on the sheet: D1, D2, D6, J1, R2, R3, R4, RN1, RN10, RN2, RN3, RN4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
