File: Control_board/Control_board.kicad_sch (KiCad schematic)
At the start: 99 parts, among them J1 Conn_02x32_Odd_Even, J1 ICSP, J3 Conn_01x02, SW1 SW_Push, SW2 SW_Push, SW3 SW_Push, SW4 SW_Push, U1 74LS74, U10 27C512, U11 ATtiny85-20P, U12 74LS74, U2 74LS74, U3 74LS273, U4 74LS373, U5 74LS192, U6 74LS373, U7 27C512, U8 27C512, U9 27C512

Commit message: Memory board
Connections:
- net +5V: now also U5.4 (DOWN)
- net GND: no longer U5.4 (DOWN)
Changed lines of the file:
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@@
 (kicad_sch (version 20230121) (generator eeschema)
   (paper "A2")
+  (junction (at 68.58 212.09) (diameter 0) (color 0 0 0 0)
+  )
   (junction (at 355.6 71.12) (diameter 0) (color 0 0 0 0)
   )
@@
   (junction (at 303.53 217.17) (diameter 0) (color 0 0 0 0)
   )
-  (junction (at 53.34 229.87) (diameter 0) (color 0 0 0 0)
-  )
   (junction (at 228.6 156.21) (diameter 0) (color 0 0 0 0)
   )
@@
   (junction (at 234.95 283.21) (diameter 0) (color 0 0 0 0)
   )
-  (junction (at 53.34 242.57) (diameter 0) (color 0 0 0 0)
-  )
   (junction (at 68.58 326.39) (diameter 0) (color 0 0 0 0)
   )
@@
   (junction (at 68.58 285.75) (diameter 0) (color 0 0 0 0)
   )
-  (junction (at 53.34 224.79) (diameter 0) (color 0 0 0 0)
+  (junction (at 50.8 227.33) (diameter 0) (color 0 0 0 0)
   )
   (junction (at 241.3 227.33) (diameter 0) (color 0 0 0 0)
@@
   (junction (at 246.38 138.43) (diameter 0) (color 0 0 0 0)
   )
+  (junction (at 50.8 229.87) (diameter 0) (color 0 0 0 0)
+  )
   (junction (at 355.6 119.38) (diameter 0) (color 0 0 0 0)
   )
@@
   (junction (at 271.78 280.67) (diameter 0) (color 0 0 0 0)
   )
+  (junction (at 50.8 224.79) (diameter 0) (color 0 0 0 0)
+  )
   (junction (at 227.33 308.61) (diameter 0) (color 0 0 0 0)
   )
@@
   (junction (at 233.68 151.13) (diameter 0) (color 0 0 0 0)
   )
-  (junction (at 53.34 227.33) (diameter 0) (color 0 0 0 0)
-  )
   (junction (at 241.3 143.51) (diameter 0) (color 0 0 0 0)
   )
@@
     (stroke (width 0) (type default))
   )
-  (wire (pts (xy 53.34 227.33) (xy 53.34 229.87))
+  (wire (pts (xy 50.8 227.33) (xy 50.8 229.87))
     (stroke (width 0) (type default))
   )
@@
     (stroke (width 0) (type default))
   )
-  (wire (pts (xy 53.34 242.57) (xy 53.34 247.65))
-    (stroke (width 0) (type default))
-  )
   (wire (pts (xy 38.1 334.01) (xy 60.96 334.01))
     (stroke (width 0) (type default))
@@
     (stroke (width 0) (type default))
   )
+  (wire (pts (xy 50.8 229.87) (xy 55.88 229.87))
+    (stroke (width 0) (type default))
+  )
   (wire (pts (xy 209.55 232.41) (xy 246.38 232.41))
     (stroke (width 0) (type default))
@@
     (stroke (width 0) (type default))
   )
-  (wire (pts (xy 53.34 224.79) (xy 53.34 227.33))
+  (wire (pts (xy 50.8 224.79) (xy 50.8 227.33))
     (stroke (width 0) (type default))
   )
@@
     (stroke (width 0) (type default))
   )
-  (wire (pts (xy 55.88 222.25) (xy 53.34 222.25))
+  (wire (pts (xy 55.88 222.25) (xy 50.8 222.25))
     (stroke (width 0) (type default))
   )
@@
     (stroke (width 0) (type default))
   )
+  (wire (pts (xy 50.8 227.33) (xy 55.88 227.33))
+    (stroke (width 0) (type default))
+  )
   (wire (pts (xy 255.27 293.37) (xy 257.81 293.37))
     (stroke (width 0) (type default))
@@
     (stroke (width 0) (type default))
   )
-  (wire (pts (xy 55.88 224.79) (xy 53.34 224.79))
-    (stroke (width 0) (type default))
-  )
   (bus (pts (xy 167.64 64.77) (xy 167.64 67.31))
     (stroke (width 0) (type default))
@@
     (stroke (width 0) (type default))
   )
-  (wire (pts (xy 53.34 242.57) (xy 55.88 242.57))
-    (stroke (width 0) (type default))
-  )
   (wire (pts (xy 209.55 300.99) (xy 234.95 300.99))
     (stroke (width 0) (type default))
@@
     (stroke (width 0) (type default))
   )
+  (wire (pts (xy 53.34 212.09) (xy 68.58 212.09))
+    (stroke (width 0) (type default))
+  )
   (wire (pts (xy 50.8 347.98) (xy 50.8 350.52))
     (stroke (width 0) (type default))
@@
     (stroke (width 0) (type default))
   )
+  (wire (pts (xy 53.34 242.57) (xy 53.34 212.09))
+    (stroke (width 0) (type default))
+  )
   (wire (pts (xy 245.11 321.31) (xy 245.11 323.85))
     (stroke (width 0) (type default))
@@
     (stroke (width 0) (type default))
   )
-  (wire (pts (xy 55.88 229.87) (xy 53.34 229.87))
-    (stroke (width 0) (type default))
-  )
   (wire (pts (xy 170.18 105.41) (xy 189.23 105.41))
     (stroke (width 0) (type default))
@@
     (stroke (width 0) (type default))
   )
-  (wire (pts (xy 53.34 229.87) (xy 53.34 242.57))
+  (wire (pts (xy 50.8 229.87) (xy 50.8 247.65))
     (stroke (width 0) (type default))
   )
@@
     (stroke (width 0) (type default))
   )
-  (wire (pts (xy 53.34 222.25) (xy 53.34 224.79))
+  (wire (pts (xy 50.8 222.25) (xy 50.8 224.79))
     (stroke (width 0) (type default))
   )
@@
     (stroke (width 0) (type default))
   )
+  (wire (pts (xy 68.58 209.55) (xy 68.58 212.09))
+    (stroke (width 0) (type default))
+  )
   (wire (pts (xy 82.55 111.76) (xy 76.2 111.76))
     (stroke (width 0) (type default))
@@
     (stroke (width 0) (type default))
   )
+  (wire (pts (xy 50.8 224.79) (xy 55.88 224.79))
+    (stroke (width 0) (type default))
+  )
   (wire (pts (xy 189.23 171.45) (xy 170.18 171.45))
     (stroke (width 0) (type default))
@@
     (stroke (width 0) (type default))
   )
+  (wire (pts (xy 55.88 242.57) (xy 53.34 242.57))
+    (stroke (width 0) (type default))
+  )
   (wire (pts (xy 189.23 74.93) (xy 170.18 74.93))
     (stroke (width 0) (type default))
@@
     (stroke (width 0) (type default))
   )
-  (wire (pts (xy 55.88 227.33) (xy 53.34 227.33))
-    (stroke (width 0) (type default))
-  )
   (wire (pts (xy 255.27 308.61) (xy 257.81 308.61))
     (stroke (width 0) (type default))
@@
   )
   (text "Count occurs on rising edge clock, latch is \nonly nescessary for the asynchronous resets"
-    (at 33.02 203.2 0)
+    (at 17.78 207.01 0)
     (effects (font (size 1.27 1.27)) (justify left bottom))
   )
@@
     )
   )
-  (symbol (lib_id "power:+5V") (at 68.58 212.09 0) (unit 1)
+  (symbol (lib_id "power:+5V") (at 68.58 209.55 0) (unit 1)
     (in_bom yes) (on_board yes) (dnp no) (fields_autoplaced)
-    (property "Reference" "#PWR0103" (at 68.58 215.9 0)
+    (property "Reference" "#PWR0103" (at 68.58 213.36 0)
       (effects (font (size 1.27 1.27)) hide)
     )
-    (property "Value" "+5V" (at 68.58 207.01 0)
+    (property "Value" "+5V" (at 68.58 204.47 0)
       (effects (font (size 1.27 1.27)))
     )
-    (property "Footprint" "" (at 68.58 212.09 0)
+    (property "Footprint" "" (at 68.58 209.55 0)
       (effects (font (size 1.27 1.27)) hide)
     )
-    (property "Datasheet" "" (at 68.58 212.09 0)
+    (property "Datasheet" "" (at 68.58 209.55 0)
       (effects (font (size 1.27 1.27)) hide)
     )
@@
     )
   )
-  (symbol (lib_id "power:GND") (at 53.34 247.65 0) (unit 1)
+  (symbol (lib_id "power:GND") (at 50.8 247.65 0) (unit 1)
     (in_bom yes) (on_board yes) (dnp no) (fields_autoplaced)
-    (property "Reference" "#PWR0133" (at 53.34 254 0)
+    (property "Reference" "#PWR0133" (at 50.8 254 0)
       (effects (font (size 1.27 1.27)) hide)
     )
-    (property "Value" "GND" (at 53.34 252.73 0)
+    (property "Value" "GND" (at 50.8 252.73 0)
       (effects (font (size 1.27 1.27)))
     )
-    (property "Footprint" "" (at 53.34 247.65 0)
+    (property "Footprint" "" (at 50.8 247.65 0)
       (effects (font (size 1.27 1.27)) hide)
     )
-    (property "Datasheet" "" (at 53.34 247.65 0)
+    (property "Datasheet" "" (at 50.8 247.65 0)
       (effects (font (size 1.27 1.27)) hide)
     )
